File: MCU.kicad_sch (KiCad schematic)
At the start: 83 parts, among them J1 Conn_01x02_Pin, J11 Logger Connector, J12 UART Connector, J13 External UART, J14 External I2C, J15 JTAG Header, J2 Conn_01x02_Pin, J27 Conn_01x02_Pin, SW1 XRSn_button, U13 M24M01E-FMN6TP, U17 TRS3221EIPWR, U5 F280025PNS, Y2 H130B-16.000-18-3030-EXT-TR

Commit message: finished 70% of the layout, only power is remaining + matching parts with each other (analog)
Connections:
- net CH1_A: no longer R12.1, U5.80 (GPIO6)
- net CH1_B: no longer R13.1, U5.79 (GPIO14)
- net CH2_A: no longer R14.1, U5.78 (GPIO15)
- net CH2_B: no longer R15.1, U5.77 (GPIO34)
- net CH3_A: no longer R16.1, U5.76 (GPIO10)
- net CH3_B: no longer R17.1, U5.75 (GPIO9)
- net CH4_A: no longer R18.1, U5.74 (GPIO5)
- net CH4_B: no longer R19.1
- net CH5_A: no longer R11.1, TP62.1, U5.62 (GPIO1)
- net CH5_B: no longer R4.1, TP61.1, U5.63 (GPIO0)
- net CH6_A: no longer R6.1, U5.64 (GPIO40)
- net CH6_B: no longer R7.1, U5.65 (GPIO23)
- net CH7_A: no longer R10.1, U5.66 (GPIO41)
- net CH7_B: no longer R9.1, U5.67 (GPIO22)
- net CH8_A: no longer R8.1, U5.68 (GPIO7)
- net CH8_B: no longer R5.1
- new net CH1_A_MCU: R12.1, U5.80 (GPIO6)
- new net CH1_B_MCU: R13.1, U5.79 (GPIO14)
- new net CH2_A_MCU: R14.1, U5.78 (GPIO15)
- new net CH2_B_MCU: R15.1, U5.77 (GPIO34)
- new net CH3_A_MCU: R16.1, U5.76 (GPIO10)
- new net CH3_B_MCU: R17.1, U5.75 (GPIO9)
- new net CH4_A_MCU: R18.1, U5.74 (GPIO5)
- new net CH4_B_MCU: R19.1
- new net CH5_A_MCU: R11.1, TP62.1, U5.62 (GPIO1)
- new net CH5_B_MCU: R4.1, TP61.1, U5.63 (GPIO0)
- new net CH6_A_MCU: R6.1, U5.64 (GPIO40)
- new net CH6_B_MCU: R7.1, U5.65 (GPIO23)
- new net CH7_A_MCU: R10.1, U5.66 (GPIO41)
- new net CH7_B_MCU: R9.1, U5.67 (GPIO22)
- new net CH8_A_MCU: R8.1, U5.68 (GPIO7)
- new net CH8_B_MCU: R5.1
Other:
- moved on the sheet: R12, R13, R14, R15, R16, R17, R18, R19
