File: Ultrasound_NDT.kicad_pcb (KiCad board)
At the start: 6 copper layers, 100 x 100 mm, 371 parts, among them J1 Conn_01x02_Pin, J10 CONSMA002-SMD, J11 Logger Connector, J12 UART Connector, J13 External UART, J14 External I2C, J15 JTAG Header, J16 Conn_02x04_Odd_Even, J17 Input Power, J18 Conn_01x02_Pin, J19 Conn_01x02_Pin, J2 Conn_01x02_Pin, J20 Conn_01x02_Pin, J21 Conn_01x02_Pin, J22 Conn_01x02_Pin, J23 Conn_01x02_Pin, J24 Conn_01x02_Pin, J25 Conn_01x02_Pin, J26 Spectrography Power, J27 Conn_01x02_Pin, J28 Conn_02x04_Odd_Even, J3 CONSMA002-SMD, J4 CONSMA002-SMD, J5 CONSMA002-SMD, J6 CONSMA002-SMD, J7 CONSMA002-SMD, J8 CONSMA002-SMD, J9 CONSMA002-SMD, SW1 XRSn_button, U1 AD8334ACPZ, U10 TLV9354IDR, U11 TLV9354IDR, U12 TPS63700DRCR, U13 M24M01E-FMN6TP, U14 LDL212PU50R, U15 AZ1117CH2-3.3, U16 AZ1117CH2-3.3, U17 TRS3221EIPWR, U18 BZX84C3V3TS-7-F, U19 BZX84C3V3TS-7-F, U2 DSC1001DI2-125.0000T, U20 BZX84C3V3TS-7-F, U22 ESD7C3.3DT5G, U23 ESD7C3.3DT5G, U3 MAX14808ETK_, U4 AD8334ACPZ, U5 F280025PNS, U6 REF3030, U7 MIC920YC5-TR, U8 TLV9354IDR, U9 TLV9354IDR, Y2 H130B-16.000-18-3030-EXT-TR

Commit message: Several finishing updates to fit stocks & changed SMA from SMD to THT, updated schematics too
Parts:
- removed J10, J3, J4, J5, J6, J7, J8, J9: CONSMA002-SMD, CONSMA002-SMD:TE_CONSMA002-SMD
- added J301: 5-1814400-1, digikey-footprints:RF_SMA_RightAngle_5-1814400-1, F.Cu at (79.2, 39.4)
- added J302: 5-1814400-1, digikey-footprints:RF_SMA_RightAngle_5-1814400-1, F.Cu at (88.8, 39.5)
- added J303: 5-1814400-1, digikey-footprints:RF_SMA_RightAngle_5-1814400-1, F.Cu at (97.8, 39.4)
- added J304: 5-1814400-1, digikey-footprints:RF_SMA_RightAngle_5-1814400-1, F.Cu at (107.2, 39.4)
- added J305: 5-1814400-1, digikey-footprints:RF_SMA_RightAngle_5-1814400-1, F.Cu at (116.7, 39.4)
- added J306: 5-1814400-1, digikey-footprints:RF_SMA_RightAngle_5-1814400-1, F.Cu at (135.0, 39.5)
- added J307: 5-1814400-1, digikey-footprints:RF_SMA_RightAngle_5-1814400-1, F.Cu at (125.8, 39.5)
- added J308: 5-1814400-1, digikey-footprints:RF_SMA_RightAngle_5-1814400-1, F.Cu at (144.2, 39.4)
- R141: value 1k -> 500R
- Y2: footprint KiCad:H130B16000183030EXTTR -> H130B-16.000-18-3030-EXT-TR:H130B16000183030EXTTR
Connections:
- PS1 pad 4_1: +7V -> (no net)
- PS1 pad 4_2: +7V -> (no net)
- PS1 pad 4_3: +7V -> (no net)
- PS1 pad 4_4: +7V -> (no net)
- PS1 pad 4_5: +7V -> (no net)
- PS1 pad 4_6: +7V -> (no net)
- PS3 pad 4_1: +5V_PULSE -> (no net)
- PS3 pad 4_2: +5V_PULSE -> (no net)
- PS3 pad 4_3: +5V_PULSE -> (no net)
- PS3 pad 4_4: +5V_PULSE -> (no net)
- PS3 pad 4_5: +5V_PULSE -> (no net)
- PS3 pad 4_6: +5V_PULSE -> (no net)
- U12 pad 12: GND -> (no net)
- U12 pad 13: GND -> (no net)
- U12 pad 14: GND -> (no net)
- U12 pad 15: GND -> (no net)
- Y2 pad 2: unconnected-(Y2-NC_1-Pad2) -> GND
- Y2 pad 4: unconnected-(Y2-NC_2-Pad4) -> GND
Routing:
- net /Main MCU Section/AFE_GAIN_B1: vias 2 -> 1
- net /Main MCU Section/AFE_GAIN_B2: vias 2 -> 1
- net +5V_PULSE: vias 12 -> 6
Other:
- board text added: "Hear what cannot be seen"

Commit message: updated manufacturing files
Parts:
- moved J18 11.2 mm to (68.1, 47.2)
- moved J301 11.0 mm to (68.2, 39.4)
- moved J308 10.2 mm to (154.5, 39.4)
- moved J25 10.1 mm to (154.4, 47.2)
- moved J302 8.23 mm to (80.5, 39.4)
- moved J19 8.00 mm to (80.8, 47.2)
- moved J306 7.05 mm to (142.0, 39.4), turned to 0 degrees
- moved J24 6.77 mm to (142.0, 47.2)
- moved J20 5.21 mm to (92.7, 47.2)
- moved J303 5.13 mm to (92.7, 39.4)
- moved TP8 4.96 mm to (136.4, 78.0), turned to 105 degrees
- moved J23 4.06 mm to (129.8, 47.2)
- moved J307 4.05 mm to (129.8, 39.4), turned to 0 degrees
- moved J304 2.03 mm to (105.2, 39.4)
- moved J21 1.76 mm to (105.4, 47.2)
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Connections:
- PS1 pad 4_1: (no net) -> +7V
- PS1 pad 4_2: (no net) -> +7V
- PS1 pad 4_3: (no net) -> +7V
- PS1 pad 4_4: (no net) -> +7V
- PS1 pad 4_5: (no net) -> +7V
- PS1 pad 4_6: (no net) -> +7V
- PS1 pad 5_1: (no net) -> unconnected-(PS1-SW-Pad5)
- PS1 pad 5_2: (no net) -> unconnected-(PS1-SW-Pad5)
- PS1 pad 5_3: (no net) -> unconnected-(PS1-SW-Pad5)
- PS1 pad 5_4: (no net) -> unconnected-(PS1-SW-Pad5)
- PS1 pad 5_5: (no net) -> unconnected-(PS1-SW-Pad5)
- PS1 pad 5_6: (no net) -> unconnected-(PS1-SW-Pad5)
- PS3 pad 4_1: (no net) -> +5V_PULSE
- PS3 pad 4_2: (no net) -> +5V_PULSE
- PS3 pad 4_3: (no net) -> +5V_PULSE
- PS3 pad 4_4: (no net) -> +5V_PULSE
- PS3 pad 4_5: (no net) -> +5V_PULSE
- PS3 pad 4_6: (no net) -> +5V_PULSE
- PS3 pad 5_1: (no net) -> unconnected-(PS3-SW-Pad5)
- PS3 pad 5_2: (no net) -> unconnected-(PS3-SW-Pad5)
- PS3 pad 5_3: (no net) -> unconnected-(PS3-SW-Pad5)
- PS3 pad 5_4: (no net) -> unconnected-(PS3-SW-Pad5)
- PS3 pad 5_5: (no net) -> unconnected-(PS3-SW-Pad5)
- PS3 pad 5_6: (no net) -> unconnected-(PS3-SW-Pad5)
- U12 pad 12: (no net) -> GND
- U12 pad 13: (no net) -> GND
- U12 pad 14: (no net) -> GND
- U12 pad 15: (no net) -> GND
Routing:
- net +12V_VFD: track 36.3 -> 48.7 mm, vias 3 -> 5
- net /Pulsing Section/HV_OUT8: track 44.8 -> 54.3 mm
- net /Pulsing Section/HV_OUT1: track 45.2 -> 53.8 mm
- net /Pulsing Section/HV_OUT2: track 35.1 -> 43.4 mm
- net /Pulsing Section/HV_OUT7: track 37.1 -> 42.7 mm
- net GND: track 72.5 -> 67.4 mm, vias 236 -> 314
- net /Pulsing Section/HV_OUT3: track 29.1 -> 33.6 mm
- net /Pulsing Section/HV_OUT6: track 28.3 -> 32.3 mm
- net /Pulsing Section/TR8: track 29.1 -> 26.0 mm
- net /Receiving Section/HILO_A: track 15.8 -> 18.1 mm
- net HV_OUT_TAP: track 21.7 -> 22.6 mm
- net /Receiving Section/ADC5_H: track 12.8 -> 13.5 mm
- net /Receiving Section/ADC5_L: track 15.8 -> 16.3 mm
- net (no net): vias 0 -> 1
